Commit message: Add setup notes, update gripper parameters, and implement gripper rendering script

File: urdf/gripper/robot.urdf (robot description, URDF)
Before this commit: robot gripper, 3 links, 2 joints
Joints:
- joint l: limit lower=-1 upper=1 effort=10 velocity=10 -> lower=0.0058 upper=0.0156 effort=10 velocity=10
- joint r: limit lower=-1 upper=1 effort=10 velocity=10 -> lower=0.0058 upper=0.0156 effort=10 velocity=10
